File: hardware/score_board.sch (KiCad schematic (older format))
At the start: 59 parts, among them J1 BATT, J2 AVR-ISP-6, J3 External Power, SW1 Battery Power, SW2 C, SW3 A, SW4 B, SW5 RESET, U1 ATtiny13A-SSU, U2 74HC595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

Commit message: Fix some kicad libraries issues
Parts:
- J2: symbol Connector_Specialized:AVR-ISP-6 -> Connector:AVR-ISP-6
- MK1, MK2, MK3, MK4: symbol Mechanical:Mounting_Hole -> Mechanical:MountingHole
Changed lines of the file:
@@
-EESchema Schematic File Version 4
+EESchema Schematic File Version 5
 LIBS:score_board-cache
-EELAYER 26 0
+EELAYER 29 0
 EELAYER END
 $Descr A4 11693 8268
@@
 Date "2018-05-04"
 Rev "1"
-Comp "68. PS Lvíčata"
+Comp "Radovan Blažek"
 Comment1 ""
 Comment2 ""
@@
 	3150 7100 2900 7100
 $Comp
-L Mechanical:Mounting_Hole MK1
+L Mechanical:MountingHole MK1
 U 1 1 5ADAAA61
 P 6200 6900
@@
 $EndComp
 $Comp
-L Mechanical:Mounting_Hole MK2
+L Mechanical:MountingHole MK2
 U 1 1 5ADAAD50
 P 6200 7100
@@
 $EndComp
 $Comp
-L Mechanical:Mounting_Hole MK3
+L Mechanical:MountingHole MK3
 U 1 1 5ADAAD80
 P 6200 7300
@@
 $EndComp
 $Comp
-L Mechanical:Mounting_Hole MK4
+L Mechanical:MountingHole MK4
 U 1 1 5ADAADB2
 P 6200 7500
@@
 	6050 3150 6050 3550
 Connection ~ 6050 3550
-$Comp
-L Connector_Specialized:AVR-ISP-6 J2
-U 1 1 5AE2B5FD
-P 1300 7000
-F 0 "J2" H 1020 7096 50  0000 R CNN
-F 1 "AVR-ISP-6" H 1020 7005 50  0000 R CNN
-F 2 "Connector_PinHeader_2.54mm:PinHeader_2x03_P2.54mm_Vertical_SMD" V 1050 7050 50  0001 C CNN
-F 3 "" H 25  6450 50  0001 C CNN
-	1    1300 7000
-	1    0    0    -1
-$EndComp
 $Comp
 L power:+3.3V #PWR0111
@@
 Wire Wire Line
 	7450 3700 7650 3700
+$Comp
+L Connector:AVR-ISP-6 J2
+U 1 1 5AE2B5FD
+P 1300 7000
+F 0 "J2" H 1020 7096 50  0000 R CNN
+F 1 "AVR-ISP-6" H 1020 7005 50  0000 R CNN
+F 2 "Connector_PinHeader_2.54mm:PinHeader_2x03_P2.54mm_Vertical_SMD" V 1050 7050 50  0001 C CNN
+F 3 "" H 25  6450 50  0001 C CNN
+	1    1300 7000
+	1    0    0    -1
+$EndComp
 $EndSCHEMATC
